File: pcb/Laptreus-v1/Laptreus-v1.kicad_pcb (KiCad board)
At the start: 2 copper layers, 283 x 100 mm, 102 parts, among them J1 Conn_01x16, J2 Conn_01x12, SW1 _, SW10 L, SW11 ., SW12 DOWN, SW13 I, SW14 K, SW15 ,, SW16 LEFT, SW17 U, SW18 J, SW19 M, SW2 ", SW20 ENTER/RAISE, SW21 Y, SW22 H, SW23 N, SW24 SPACE, SW25 T, SW26 G, SW27 B, SW28 SHIFT, SW29 R, SW3 ENTER, SW30 F, SW31 V, SW32 BKSP/LOWER, SW33 E, SW34 D, SW35 C, SW36 CMD, SW37 W, SW38 S, SW39 X, SW4 RIGHT, SW40 OPT/TAB, SW41 Q, SW42 A, SW43 Z, SW44 CTRL/GRV, SW47 HYPER, SW48 SHIFT, SW49 ESC, SW5 P, SW50 TAB, SW6 ;, SW7 /, SW8 UP, SW9 O

Commit message: Adding first attempts at laptreus v2
Parts:
- added FID: FIDUCIAL, hole:FIDUCIAL, B.Cu at (92.6, 144.5)
- added FID: FIDUCIAL, hole:FIDUCIAL, B.Cu at (371.0, 57.1)
- added HOLE: VAL**, hole:PKRH, F.Cu at (349.3, 81.4)
- added HOLE: VAL**, hole:PKRH, F.Cu at (279.8, 138.7)
- added HOLE: VAL**, hole:PKRH, F.Cu at (217.5, 100.5)
- added HOLE: VAL**, hole:PKRHC, F.Cu at (114.5, 81.4)
- added HOLE: VAL**, hole:PKRHSL, F.Cu at (90.7, 110.0)
- added HOLE: VAL**, hole:PKRHSL, F.Cu at (372.8, 110.0)
- added J1: MINI, usb:67503, B.Cu at (107.5, 53.5)
- added S0: DTSM-6, dtsm:KSEM31GLFS, B.Cu at (118.4, 101.7)
Routing:
- net (no net): track 0.00 -> 3.39 mm, vias 0 -> 1
Other:
- board size 283 x 100 mm -> 285 x 100 mm
