File: pcb/Laptreus-v2/Laptreus-v2.sch (KiCad schematic (older format))
At the start: 105 parts, among them J1 Conn_01x16, J2 Conn_01x12, SW1 TAB, SW10 O, SW11 P, SW12 BKSP, SW13 ESC, SW14 A, SW15 S, SW16 D, SW17 F/LOWER, SW18 G, SW19 H, SW2 Q, SW20 J/RAISE, SW21 K, SW22 L, SW23 ;, SW24 \", SW25 SHIFT, SW26 Z, SW27 X, SW28 C, SW29 V, SW3 W, SW30 B, SW31 N, SW32 M, SW33 ,, SW34 ., SW35 /, SW36 ENTER, SW37 HYPER, SW38 CTRL/GRV, SW39 ALT/TAB, SW4 E, SW40 CMD, SW41 BKSP/LIFT, SW42 SHIFT, SW43 SPACE, SW44 ENTER/LIFT, SW45 LEFT, SW46 DOWN, SW47 UP, SW48 RIGHT, SW49 SPECIAL, SW5 R, SW50 SPECIAL, SW6 T, SW7 Y, SW8 U, SW9 I

Commit message: Adding first attempts at laptreus v2
Parts:
- removed D1, D12, D13, D24, D25, D36, D37, D48: DIODE, Laptreus v2 Footprints:Diode-dual, symbol Diode:1N4148
- removed J1: Conn_01x16, Connector_PinHeader_2.54mm:PinHeader_1x16_P2.54mm_Vertical, symbol Connector_Generic:Conn_01x16
- removed J2: Conn_01x12, Connector_PinHeader_2.54mm:PinHeader_1x12_P2.54mm_Vertical, symbol Connector_Generic:Conn_01x12
- removed SW1: TAB, Laptreus v2 Footprints:Hybrid_Kailh_MX_Socket_Through_Hole, symbol Switch:SW_Push
- removed SW12: BKSP, Laptreus v2 Footprints:Hybrid_Kailh_MX_Socket_Through_Hole, symbol Switch:SW_Push
- removed SW13: ESC, Laptreus v2 Footprints:Hybrid_Kailh_MX_Socket_Through_Hole, symbol Switch:SW_Push
- removed SW24: \", Laptreus v2 Footprints:Hybrid_Kailh_MX_Socket_Through_Hole, symbol Switch:SW_Push
- removed SW25: SHIFT, Laptreus v2 Footprints:Hybrid_Kailh_MX_Socket_Through_Hole, symbol Switch:SW_Push
- removed SW36: ENTER, Laptreus v2 Footprints:Hybrid_Kailh_MX_Socket_Through_Hole, symbol Switch:SW_Push
- removed SW37: HYPER, Laptreus v2 Footprints:Hybrid_Kailh_MX_Socket_Through_Hole, symbol Switch:SW_Push
- removed SW48: RIGHT, Laptreus v2 Footprints:Hybrid_Kailh_MX_Socket_Through_Hole, symbol Switch:SW_Push
- added C1, C3, C5: 10µF, Adafruit Feather 32u4 Bluefruit LE:_0805MP, symbol Adafruit-parts:CAP_CERAMIC0805-NOOUTLINE
- added C10, C11, C12, C13, C14, C15, C8, C9: 1uF, Adafruit Feather 32u4 Bluefruit LE:_0805MP, symbol Adafruit-parts:C-EUC0805
- added C2, C4, C6: 1uF, Adafruit Feather 32u4 Bluefruit LE:_0805MP, symbol Adafruit-parts:CAP_CERAMIC0603_NO
- added C7: 10uF, Adafruit Feather 32u4 Bluefruit LE:_0805MP, symbol Adafruit-parts:CAP_CERAMIC_0805MP
- added CHG1: ORANGE, Adafruit Feather 32u4 Bluefruit LE:CHIPLED_0805_NOOUTLINE, symbol Adafruit-parts:LED0805_NOOUTLINE
- added D1: MBR120, Adafruit Feather 32u4 Bluefruit LE:SOD-123, symbol Adafruit-parts:DIODE-SCHOTTKYSOD-123
- added D12, L1: RED, Adafruit Feather 32u4 Bluefruit LE:CHIPLED_0805_NOOUTLINE, symbol Adafruit-parts:LED0805_NOOUTLINE
- added D13: BLUE, Adafruit Feather 32u4 Bluefruit LE:CHIPLED_0805_NOOUTLINE, symbol Adafruit-parts:LED0805_NOOUTLINE
- added IC1: ATMEGA32U4-MU, Adafruit Feather 32u4 Bluefruit LE:TQFN44_7MM, symbol Adafruit-parts:ATMEGA32U4-MU
- added JP1, JP2, JP3, JP4: PINHD-1X1CB, Adafruit NeoPixel Ring 12:1X01-CLEANBIG, symbol Adafruit-parts:PINHD-1X1CB
- added LED1, LED10, LED11, LED12, LED2, LED3, LED4, LED5, LED6, LED7, LED8, LED9: WS28115050, Adafruit NeoPixel Ring 12:WS28115050, symbol Adafruit-parts:WS28115050
- added R1: 1K, Adafruit Feather 32u4 Bluefruit LE:_0805MP, symbol Adafruit-parts:RESISTOR_0603_NOOUT
- added R10, R6, R7: 2.2K, Adafruit Feather 32u4 Bluefruit LE:_0805MP, symbol Adafruit-parts:RESISTOR_0603_NOOUT
- added R2, R4, R5: 100K, Adafruit Feather 32u4 Bluefruit LE:_0805MP, symbol Adafruit-parts:RESISTOR_0603_NOOUT
- added R3: 10K\\, Adafruit Feather 32u4 Bluefruit LE:_0805MP, symbol Adafruit-parts:RESISTOR_0603_NOOUT
- added R8, R9: 22, Adafruit Feather 32u4 Bluefruit LE:_0805MP, symbol Adafruit-parts:RESISTOR_0603_NOOUT
- added TP1: SWCLK, Adafruit Feather 32u4 Bluefruit LE:PAD-1.5X2.0, symbol Adafruit-parts:TESTPOINT1.5X2.0MM_NOCREAM
- added TP2, TP3: SWDIO, Adafruit Feather 32u4 Bluefruit LE:PAD-1.5X2.0, symbol Adafruit-parts:TESTPOINT1.5X2.0MM_NOCREAM
- added U1: MCP73831T-2ACI/OT, Adafruit Feather 32u4 Bluefruit LE:SOT23-5, symbol Adafruit-parts:MCP73831_2
- added U2: SPX3819-3.3, Adafruit Feather 32u4 Bluefruit LE:SOT23-5, symbol Adafruit-parts:VREG_SOT23-5
- added U3: MBT40, Adafruit Feather 32u4 Bluefruit LE:BLE_MODULE_RAYTAC_MDBT40, symbol Adafruit-parts:NRF51822_MODULE_MDBT40
- added X1: JSTPH, Adafruit Feather 32u4 Bluefruit LE:JSTPH2, symbol Adafruit-parts:CON_JST_PH_2PIN
- added X2: microUSB, Adafruit Feather 32u4 Bluefruit LE:4UCONN_20329_V2, symbol Adafruit-parts:USB_MICRO_20329_V2
- added Y1: 8MHz, Adafruit Feather 32u4 Bluefruit LE:RESONATOR-SMD, symbol Adafruit-parts:RESONATORSMD
- SW41: value BKSP/LIFT -> SHIFT
- SW42: value SHIFT -> BKSP/LIFT
- SW43: value SPACE -> ENTER/LIFT
- SW44: value ENTER/LIFT -> SPACE
- SW_RESET2: footprint Laptreus-v1:Hybrid_Kailh_MX_Socket_Through_Hole -> Laptreus v2 Footprints:Hybrid_Kailh_MX_Socket_Through_Hole
Connections:
- net labels added: +3V3, 13, 4_SWDIO/RST, 7_BLE_IRQ, 8_BLE_CS, 9, AREF, CONNECTED, DCC, DEC2, DFU, EN, FCTRYRST, MISO, MODE, MOSI, SCK, SWCLK, VBAT, VBUS, VDD
- net labels removed: +5V, Enable
- wire segments 399 -> 585
- no-connect marks 10 -> 29
Other:
- note added: "1.0K = 1000mA"
- note added: "10K = 100mA"
- note added: "2.0K = 500mA"
- note added: "5.0K = 200mA"
- note added: "ATMEGA32U4 MCU"
- note added: "BLUEFRUIT LE MODULE (nRF51)"
- note added: "LIPO & CHARGING"
- note added: "POWER AND FILTERING"
- note added: "POWER SWITCH"
- note added: "RESET BUTTONS"
- note removed: "Header\nPins\n"
- note removed: "Power\nSwitch"
- note removed: "Reset\nButtons"
- moved on the sheet: D10, D11, D14, D15, D16, D17, D18, D19, D2, D20, D21, D22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

Commit message: switches aligned, leds circled
Parts:
- removed R10: 2.2K, Adafruit Feather 32u4 Bluefruit LE:_0805MP, symbol Adafruit-parts:RESISTOR_0603_NOOUT
- removed R8, R9: 22, Adafruit Feather 32u4 Bluefruit LE:_0805MP, symbol Adafruit-parts:RESISTOR_0603_NOOUT
- removed X2: microUSB, Adafruit Feather 32u4 Bluefruit LE:4UCONN_20329_V2, symbol Adafruit-parts:USB_MICRO_20329_V2
- added D1, D12, D13, D24, D25, D36, D37, D48: DIODE, Laptreus v2 Footprints:Diode-dual, symbol Diode:1N4148
- added F1: Polyfuse, Adafruit Feather 32u4 Bluefruit LE:0805-NO, symbol Device:Polyfuse
- added H1: B7, Adafruit NeoPixel Ring 12:1X01-CLEANBIG, symbol Connector_Generic:Conn_01x01
- added H2: GND, Adafruit NeoPixel Ring 12:1X01-CLEANBIG, symbol Connector_Generic:Conn_01x01
- added H3: +5v, Adafruit NeoPixel Ring 12:1X01-CLEANBIG, symbol Connector_Generic:Conn_01x01
- added H4: B0, Adafruit NeoPixel Ring 12:1X01-CLEANBIG, symbol Connector_Generic:Conn_01x01
- added J1: HRO-TYPE-C-31-M-12, Laptreus v2 Footprints:HRO-TYPE-C-31-M-12, symbol Laptreus-v2-rescue:HRO-TYPE-C-31-M-12-Type-C
- added J2: ISP, Laptreus v2 Footprints:isp_standard, symbol Connector_Generic:Conn_02x03_Odd_Even
- added R10: 10k, Adafruit Feather 32u4 Bluefruit LE:0805-NO, symbol Device:R
- added R11, R12: 5.1k, Adafruit Feather 32u4 Bluefruit LE:0805-NO, symbol Device:R
- added R8, R9: 22, Adafruit Feather 32u4 Bluefruit LE:0805-NO, symbol Device:R
- added S1, S2, S3, S6: Screw, Laptreus v2 Footprints:PKRH, symbol Connector:Screw_Terminal_01x01
- added S4, S5: Screw, Laptreus v2 Footprints:PKRHSL, symbol Connector:Screw_Terminal_01x01
- added S7, S8, S9: Tofu screw, Laptreus v2 Footprints:PKRH, symbol Connector:Screw_Terminal_01x01
- added SW1: TAB, Laptreus v2 Footprints:Hybrid_Kailh_MX_Socket_Through_Hole, symbol Switch:SW_Push
- added SW12: BKSP, Laptreus v2 Footprints:Hybrid_Kailh_MX_Socket_Through_Hole, symbol Switch:SW_Push
- added SW13: ESC, Laptreus v2 Footprints:Hybrid_Kailh_MX_Socket_Through_Hole, symbol Switch:SW_Push
- added SW24: \", Laptreus v2 Footprints:Hybrid_Kailh_MX_Socket_Through_Hole, symbol Switch:SW_Push
- added SW25: SHIFT, Laptreus v2 Footprints:Hybrid_Kailh_MX_Socket_Through_Hole, symbol Switch:SW_Push
- added SW36: ENTER, Laptreus v2 Footprints:Hybrid_Kailh_MX_Socket_Through_Hole, symbol Switch:SW_Push
- added SW37: HYPER, Laptreus v2 Footprints:Hybrid_Kailh_MX_Socket_Through_Hole, symbol Switch:SW_Push
- added SW48: RIGHT, Laptreus v2 Footprints:Hybrid_Kailh_MX_Socket_Through_Hole, symbol Switch:SW_Push
- added SW_POW_EN2: SW_SPDT, Laptreus v2 Footprints:EG1218, symbol Switch:SW_SPDT
- added U6: USBLC6-2SC6, Laptreus v2 Footprints:USBLC6-2SC6, symbol Laptreus-v2-rescue:USBLC6-2SC6-keyboard_parts
- renumbered D1 to D49, D49 to D55, D50 to D56, D12 to D60, D13 to D61
Connections:
- net EN: now also SW_POW_EN2.2 (B)
- net GND: now also H2.1 (Pin_1), J1.1 (GND), J1.12 (GND), J1.13 (SHIELD), J2.6 (Pin_6), R10.1, R11.2, R12.1, S1.1 (Pin_1), S2.1 (Pin_1), S3.1 (Pin_1), S4.1 (Pin_1), S5.1 (Pin_1), S6.1 (Pin_1), S7.1 (Pin_1), S8.1 (Pin_1), S9.1 (Pin_1), SW_POW_EN2.1 (A), U6.2 (GND)
- net MISO: now also J2.1 (Pin_1)
- net MOSI: now also J2.4 (Pin_4)
- net ROW0: now also SW1.1, SW12.1
- net ROW1: now also SW13.1, SW24.1
- net ROW2: now also SW25.1, SW36.1
- net ROW3: now also SW37.1, SW48.1
- net SCK: now also J2.3 (Pin_3)
- net VBUS: now also F1.2, J1.11 (VBUS), J1.2 (VBUS), U6.5 (VBUS)
- net at IC1.4 (D+): now also R8.1
- net at IC1.3 (D-): now also R9.2
- net COL11: now reaches IC1.22 (PD5(XCK/CTS))
- net COL11: now also D1.2 (A), D13.2 (A), D25.2 (A), D37.2 (A)
- net COL0: now reaches IC1.8 (PB0(SS))
- net COL0: now also D12.2 (A), D24.2 (A), D36.2 (A), D48.2 (A)
- new net: J1.10 (CC2), R11.1
- new net: J1.4 (CC1), R12.2
- new net: D1.1 (K), SW1.2
- new net: D13.1 (K), SW13.2
- new net: D25.1 (K), SW25.2
- new net: D37.1 (K), SW37.2
- new net: D12.1 (K), SW12.2
- new net: D24.1 (K), SW24.2
- new net: D36.1 (K), SW36.2
- new net: D48.1 (K), SW48.2
- new net: R8.2, U6.6 (I/O1)
- new net: R9.1, U6.4 (I/O2)
- new net D+: J1.6 (DP1), J1.8 (DP2), U6.1 (I/O1)
- new net D-: J1.5 (DN2), J1.7 (DN1), U6.3 (I/O2)
- new net RST: J2.5 (Pin_5)
- new net VCC: F1.1, H3.1 (Pin_1), J2.2 (Pin_2)
Other:
- note added: "POWER SWITCHES"
- note removed: "POWER SWITCH"
- moved on the sheet: C1, C10, C11, C12, C13, C14, C15, C2, C3, C4, C5, C6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

Commit message: Starting work on the atmega layout
Parts:
- removed S3: Screw, Laptreus v2 Footprints:PKRH, symbol Connector:Screw_Terminal_01x01
- added C16: 100nF, Laptreus v2 Footprints:Capacitor-0805MP, symbol Adafruit-parts:CAP_CERAMIC_0805MP
- C1, C10, C11, C12, C13, C14, C15, C2, C3, C4, C5, C6, C7, C8, C9: footprint Adafruit Feather 32u4 Bluefruit LE:_0805MP -> Laptreus v2 Footprints:Capacitor-0805MP
- F1, R10, R11, R12, R8, R9: footprint Adafruit Feather 32u4 Bluefruit LE:0805-NO -> Laptreus v2 Footprints:0805-NO
- R1, R2, R3, R4, R5, R6, R7: footprint Adafruit Feather 32u4 Bluefruit LE:_0805MP -> Laptreus v2 Footprints:0805-NO
- S1: footprint Laptreus v2 Footprints:PKRH -> Laptreus v2 Footprints:PKRH-Round
- SW12: footprint Laptreus v2 Footprints:Hybrid_Kailh_MX_Socket_Through_Hole -> Laptreus v2 Footprints:Hybrid_Kailh_MX_Socket
Connections:
- net +3V3: now also IC1.14 (VCC), IC1.24 (AVCC), IC1.44 (AVCC1), IC1.7 (VBUS); no longer C7.1, IC1.6 (UCAP)
- net GND: now also C16.1
- net VBUS: now also C16.2; no longer IC1.7 (VBUS)
- net VCC: no longer F1.1, J2.2 (Pin_2)
- new net UCAP: C7.1, IC1.6 (UCAP)
Other:
- moved on the sheet: C7, S4, S5, S6

Commit message: prep for printing v2.1 of the laptre
Parts:
- removed C1: 10µF, Laptreus v2 Footprints:Capacitor-0805MP, symbol Adafruit-parts:CAP_CERAMIC0805-NOOUTLINE
- removed C10, C11, C12, C13, C14, C15, C8, C9: 1uF, Laptreus v2 Footprints:Capacitor-0805MP, symbol Adafruit-parts:C-EUC0805
- removed C16: 100nF, Laptreus v2 Footprints:Capacitor-0805MP, symbol Adafruit-parts:CAP_CERAMIC_0805MP
- removed C2, C6: 1uF, Laptreus v2 Footprints:Capacitor-0805MP, symbol Adafruit-parts:CAP_CERAMIC0603_NO
- removed CHG1: ORANGE, Adafruit Feather 32u4 Bluefruit LE:CHIPLED_0805_NOOUTLINE, symbol Adafruit-parts:LED0805_NOOUTLINE
- removed D49: MBR120, Adafruit Feather 32u4 Bluefruit LE:SOD-123, symbol Adafruit-parts:DIODE-SCHOTTKYSOD-123
- removed D55, D56: DIODE, Laptreus v2 Footprints:Diode-dual, symbol Diode:1N4148
- removed D60: RED, Adafruit Feather 32u4 Bluefruit LE:CHIPLED_0805_NOOUTLINE, symbol Adafruit-parts:LED0805_NOOUTLINE
- removed D61: BLUE, Adafruit Feather 32u4 Bluefruit LE:CHIPLED_0805_NOOUTLINE, symbol Adafruit-parts:LED0805_NOOUTLINE
- removed H1: B7, Adafruit NeoPixel Ring 12:1X01-CLEANBIG, symbol Connector_Generic:Conn_01x01
- removed H2: GND, Adafruit NeoPixel Ring 12:1X01-CLEANBIG, symbol Connector_Generic:Conn_01x01
- removed H3: +5v, Adafruit NeoPixel Ring 12:1X01-CLEANBIG, symbol Connector_Generic:Conn_01x01
- removed H4: B0, Adafruit NeoPixel Ring 12:1X01-CLEANBIG, symbol Connector_Generic:Conn_01x01
- removed J2: ISP, Laptreus v2 Footprints:isp_standard, symbol Connector_Generic:Conn_02x03_Odd_Even
- removed JP4: PINHD-1X1CB, Adafruit NeoPixel Ring 12:1X01-CLEANBIG, symbol Adafruit-parts:PINHD-1X1CB
- removed LED1, LED10, LED11, LED12, LED2, LED3, LED4, LED5, LED6, LED7, LED8, LED9: WS28115050, Adafruit NeoPixel Ring 12:WS28115050, symbol Adafruit-parts:WS28115050
- removed R1: 1K, Laptreus v2 Footprints:0805-NO, symbol Adafruit-parts:RESISTOR_0603_NOOUT
- removed R2, R4, R5: 100K, Laptreus v2 Footprints:0805-NO, symbol Adafruit-parts:RESISTOR_0603_NOOUT
- removed R3: 10K\\, Laptreus v2 Footprints:0805-NO, symbol Adafruit-parts:RESISTOR_0603_NOOUT
- removed R6, R7: 2.2K, Laptreus v2 Footprints:0805-NO, symbol Adafruit-parts:RESISTOR_0603_NOOUT
- removed S1: Screw, Laptreus v2 Footprints:PKRH-Round, symbol Connector:Screw_Terminal_01x01
- removed S2, S6: Screw, Laptreus v2 Footprints:PKRH, symbol Connector:Screw_Terminal_01x01
- removed S4, S5: Screw, Laptreus v2 Footprints:PKRHSL, symbol Connector:Screw_Terminal_01x01
- removed S7, S8, S9: Tofu screw, Laptreus v2 Footprints:PKRH, symbol Connector:Screw_Terminal_01x01
- removed SW49, SW50: SPECIAL, Laptreus v2 Footprints:Hybrid_Kailh_MX_Socket_Through_Hole, symbol Switch:SW_Push
- removed SW_POW_EN1, SW_POW_EN2: SW_SPDT, Laptreus v2 Footprints:EG1218, symbol Switch:SW_SPDT
- removed TP1: SWCLK, Adafruit Feather 32u4 Bluefruit LE:PAD-1.5X2.0, symbol Adafruit-parts:TESTPOINT1.5X2.0MM_NOCREAM
- removed TP2, TP3: SWDIO, Adafruit Feather 32u4 Bluefruit LE:PAD-1.5X2.0, symbol Adafruit-parts:TESTPOINT1.5X2.0MM_NOCREAM
- removed U1: MCP73831T-2ACI/OT, Adafruit Feather 32u4 Bluefruit LE:SOT23-5, symbol Adafruit-parts:MCP73831_2
- removed U2: SPX3819-3.3, Adafruit Feather 32u4 Bluefruit LE:SOT23-5, symbol Adafruit-parts:VREG_SOT23-5
- removed U3: MBT40, Adafruit Feather 32u4 Bluefruit LE:BLE_MODULE_RAYTAC_MDBT40, symbol Adafruit-parts:NRF51822_MODULE_MDBT40
- removed U6: USBLC6-2SC6, Laptreus v2 Footprints:USBLC6-2SC6, symbol Laptreus-v2-rescue:USBLC6-2SC6-keyboard_parts
- removed X1: JSTPH, Adafruit Feather 32u4 Bluefruit LE:JSTPH2, symbol Adafruit-parts:CON_JST_PH_2PIN
- added BOARD1: BoardOutline, Laptreus v2 Footprints:60-percent-plus-tofu, symbol Laptreus-v2:BoardOutline
- added C2: 1µF, Laptreus v2 Footprints:Capacitor-0805MP, symbol Adafruit-parts:CAP_CERAMIC0805-NOOUTLINE
- added FID1, FID2, FID3, FID4: Fiducial, Laptreus v2 Footprints:FIDUCIAL, symbol Mechanical:Fiducial
- added R1: 1K, Laptreus v2 Footprints:0805-NO, symbol Device:R_Small
- added R13: 1K, Laptreus v2 Footprints:0805-NO, symbol Device:R
- added U6: PRTR5V0U2X, Laptreus v2 Footprints:SOT143B, symbol Power_Protection:PRTR5V0U2X
- C3: LCSC Part Number (none) -> C77073; Manufacturer (none) -> Murata; Manufacturer Part Number (none) -> GRM21BR61A106KE19L; Package (none) -> 0805; Type (none) -> Capacitor
- C4: value 1uF -> 1µF; symbol Adafruit-parts:CAP_CERAMIC0603_NO -> Adafruit-parts:CAP_CERAMIC0805-NOOUTLINE; LCSC Part Number (none) -> C77079; Manufacturer (none) -> Murata; Manufacturer Part Number (none) -> GRM21BR71C105KA01L; Package (none) -> 0805; Type (none) -> Capacitor
- C5: value 10µF -> 1µF; LCSC Part Number (none) -> C77079; Manufacturer (none) -> Murata; Manufacturer Part Number (none) -> GRM21BR71C105KA01L; Package (none) -> 0805; Type (none) -> Capacitor
- C7: value 10uF -> 1µF; LCSC Part Number (none) -> C77079; Manufacturer (none) -> Murata; Manufacturer Part Number (none) -> GRM21BR71C105KA01L; Package (none) -> 0805; Type (none) -> Capacitor
- D1, D10, D11, D12, D13, D14, D15, D16, D17, D18, D19, D2, D20, D21, D22, D23, D24, D25, D26, D27, D28, D29, D3, D30, D31, D32, D33, D34, D35, D36, D37, D38, D39, D4, D40, D41, D42, D43, D44, D45, D46, D47, D48, D5, D6, D7, D8, D9: Generic Name (none) -> 1N4148; LCSC Part Number (none) -> C109203; Manufacturer (none) -> Shikues; Manufacturer Part Number (none) -> 1N4148W; Package (none) -> SOD-123; Type (none) -> Diode
- F1: footprint Laptreus v2 Footprints:0805-NO -> Fuse:Fuse_1206_3216Metric_Pad1.42x1.75mm_HandSolder; Generic Name (none) -> PPTC Resettable Fuse; LCSC Part Number (none) -> C182310; Manufacturer (none) -> Shenzhen lanson Elec; Manufacturer Part Number (none) -> 12H1200C; Package (none) -> SMD1206; Type (none) -> Polyfuse
- IC1: value ATMEGA32U4-MU -> ATMEGA32U4; footprint Adafruit Feather 32u4 Bluefruit LE:TQFN44_7MM -> Package_QFP:TQFP-44_10x10mm_P0.8mm; symbol Adafruit-parts:ATMEGA32U4-MU -> Laptreus-v2:ATMEGA32U4-MU; LCSC Part Number (none) -> C44854; Manufacturer (none) -> Microchip Tech; Manufacturer Part Number (none) -> ATMEGA32U4-AU; Package (none) -> TQFP; Type (none) -> MCU
- J1: LCSC Part Number (none) -> C223906; Manufacturer (none) -> Korean Hroparts Elec; Manufacturer Part Number (none) -> TYPE-C-31-M-13; Type (none) -> Connector
- JP1, JP2, JP3: Type (none) -> Pin
- L1: value RED -> YELLOW; LCSC Part Number (none) -> C192671; Manufacturer (none) -> TOGIALED; Manufacturer Part Number (none) -> TJ-S2012SW8TGLC9Y-A5; Package (none) -> 0805; Type (none) -> LED
- R10: value 10k -> 1K; LCSC Part Number (none) -> C101404; Manufacturer (none) -> LIZ Elec; Manufacturer Part Number (none) -> CR0805F81001G; Package (none) -> 0805; Type (none) -> Resistor
- R11, R12: value 5.1k -> 5.1K; LCSC Part Number (none) -> C101769; Manufacturer (none) -> LIZ Elec; Manufacturer Part Number (none) -> CR0805F85101G; Package (none) -> 0805; Type (none) -> Resistor
- R8, R9: LCSC Part Number (none) -> C101576; Manufacturer (none) -> LIZ Elec; Manufacturer Part Number (none) -> CR0805F822R0G; Package (none) -> 0805; Type (none) -> Resistor
- SW1, SW2: footprint Laptreus v2 Footprints:Hybrid_Kailh_MX_Socket_Through_Hole -> Laptreus v2 Footprints:Hybrid_Kailh_MX_Socket_No_Alignment_Pad; symbol Switch:SW_Push -> Laptreus-v2:SW_Push; Manufacturer Part Number (none) -> CPG151101S11; Package (none) -> PG1511; Type (none) -> Socket
- SW10, SW11, SW13, SW14, SW15, SW16, SW17, SW18, SW19, SW20, SW21, SW22, SW23, SW24, SW25, SW26, SW27, SW28, SW29, SW3, SW30, SW31, SW32, SW33, SW34, SW35, SW36, SW37, SW38, SW39, SW4, SW40, SW41, SW42, SW43, SW44, SW45, SW46, SW47, SW48, SW5, SW6, SW7, SW8, SW9, SW_RESET2: footprint Laptreus v2 Footprints:Hybrid_Kailh_MX_Socket_Through_Hole -> Laptreus v2 Footprints:Hybrid_Kailh_MX_Socket_Through_Hole_No_Alignment_Pad; symbol Switch:SW_Push -> Laptreus-v2:SW_Push; Manufacturer Part Number (none) -> CPG151101S11; Package (none) -> PG1511; Type (none) -> Socket
- SW12: footprint Laptreus v2 Footprints:Hybrid_Kailh_MX_Socket -> Laptreus v2 Footprints:Hybrid_Kailh_MX_Socket_Through_Hole_No_Alignment_Pad; symbol Switch:SW_Push -> Laptreus-v2:SW_Push; Manufacturer Part Number (none) -> CPG151101S11; Package (none) -> PG1511; Type (none) -> Socket
- SW_RESET1: symbol Switch:SW_Push -> Laptreus-v2:SW_Push; LCSC Part Number (none) -> C231329; Manufacturer (none) -> Omron Electronics; Manufacturer Part Number (none) -> B3U-1000P; Type (none) -> SPST Switch
- Y1: LCSC Part Number (none) -> C110614; Manufacturer (none) -> Murata Electronics; Manufacturer Part Number (none) -> CSTCE8M00G15C99-R0; Package (none) -> SMD-3213-3P; Type (none) -> Ceramic Resonator
Connections:
- net 4_SWDIO/RST is gone; now on net COL5: IC1.25 (PD4(ICP1/ADC8))
- net ROW4 is gone; now on net COL8: IC1.39 (PF4(ADC4/TCK))
- net VBAT is gone; now on net +5V: C5.1
- net COL0: now also IC1.22 (PD5(XCK/CTS)); no longer IC1.8 (PB0(SS))
- net COL1: now also IC1.21 (PD3(INT3/TXD1)); no longer IC1.41 (PF0(ADC0))
- net COL10: now also IC1.37 (PF6(ADC6/TDO)); no longer IC1.26 (PD6(T1/ADC9/~OC4D))
- net COL11: now also IC1.36 (PF7(ADC7(TDI)); no longer IC1.22 (PD5(XCK/CTS))
- net COL3: now also IC1.19 (PD1(INT1/SDA)); no longer IC1.21 (PD3(INT3/TXD1))
- net COL5: no longer IC1.19 (PD1(INT1/SDA))
- net COL6: now also IC1.41 (PF0(ADC0)); no longer IC1.31 (PC6(OC3A/~OC4A))
- net COL7: now also IC1.40 (PF1(ADC1)); no longer IC1.27 (PD7(OC4D/ADC10/T0))
- net COL8: no longer IC1.30 (PB6(OC1B/OC4B/ADC13))
- net COL9: now also IC1.38 (PF5(ADC5/TMS)); no longer IC1.12 (PB7(OC0A/OC1C/RTS))
- net D+: now also R8.2, U6.2 (I/O1)
- net D-: now also R9.1, U6.3 (I/O2)
- net GND: now also JP2.1, BOARD1.1 (GND), C2.2, U6.1 (GND); no longer JP3.1
- net RESET: now also R1.1
- net ROW0: now also IC1.26 (PD6(T1/ADC9/~OC4D)); no longer IC1.36 (PF7(ADC7(TDI))
- net ROW1: now also IC1.27 (PD7(OC4D/ADC10/T0)); no longer IC1.37 (PF6(ADC6/TDO))
- net ROW2: now also IC1.30 (PB6(OC1B/OC4B/ADC13)); no longer IC1.38 (PF5(ADC5/TMS))
- net ROW3: now also IC1.31 (PC6(OC3A/~OC4A)); no longer IC1.40 (PF1(ADC1))
- net HWB: now reaches R10.2
- net HWB: now also IC1.33 (PE2(~HWB))
- net +5V: now reaches F1.1
- net +5V: now also C3.1, C4.1, IC1.14 (VCC), IC1.2 (UVCC), IC1.24 (AVCC), IC1.34 (VCC1), IC1.44 (AVCC1), IC1.7 (VBUS), JP3.1, C2.1, R1.2, U6.4 (VCC)
- net DR+: now reaches IC1.4 (D+), R8.1
- net DR-: now reaches IC1.3 (D-), R9.2
- net XTAL1: now reaches IC1.17 (XTAL1), Y1.1
- net XTAL2: now reaches IC1.16 (XTAL2), Y1.3
- net at L1.A: now also R13.1
- removed net +3V3: C3.1, C4.1, IC1.14 (VCC), IC1.24 (AVCC), IC1.33 (PE2(~HWB)), IC1.34 (VCC1), IC1.44 (AVCC1), IC1.7 (VBUS)
- net 13 renamed C7-13
- net C7-13: now also R13.2
- net 7_BLE_IRQ: no longer names the net of IC1.1 (PE6(INT.6/AIN0))
- net 8_BLE_CS renamed B4
- net 9 renamed B5-9
- net MISO renamed B3-MISO
- net MOSI renamed B2-MOSI
- net SCK renamed B1-SCK
- net VBUS renamed +5VRAW
- net VDD renamed LED_STRIP_IN
- new net B0-RST: IC1.8 (PB0(SS))
- new net B7-LED-STRIP: IC1.12 (PB7(OC0A/OC1C/RTS))
- no-connect marks 29 -> 9
Other:
- note added: "ESD Protection IC"
- note added: "FIDUCIALS"
- note added: "LED STRIP PINS"
- note added: "USB-C"
- note removed: "1.0K = 1000mA"
- note removed: "10K = 100mA"
- note removed: "2.0K = 500mA"
- note removed: "5.0K = 200mA"
- note removed: "BLUEFRUIT LE MODULE (nRF51)"
- note removed: "LIPO & CHARGING"
- note removed: "POWER SWITCHES"
- note removed: "Special\nButtons"
- moved on the sheet: C3, C4, C7, D1, D10, D11, D12, D13, D14, D15, D16, D17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
