File: pcb/Laptreus-v2/_saved_Laptreus-v2.sch (KiCad schematic (older format))
At the start: 124 parts, among them IC1 ATMEGA32U4, J1 HRO-TYPE-C-31-M-12, SW1 TAB, SW10 O, SW11 P, SW12 BKSP, SW13 ESC, SW14 A, SW15 S, SW16 D, SW17 F/LOWER, SW18 G, SW19 H, SW2 Q, SW20 J/RAISE, SW21 K, SW22 L, SW23 ;, SW24 \", SW25 SHIFT, SW26 Z, SW27 X, SW28 C, SW29 V, SW3 W, SW30 B, SW31 N, SW32 M, SW33 ,, SW34 ., SW35 /, SW36 ENTER, SW37 HYPER, SW38 CTRL/GRV, SW39 ALT/TAB, SW4 E, SW40 CMD, SW41 SHIFT, SW42 BKSP/LIFT, SW43 ENTER/LIFT, SW44 SPACE, SW45 LEFT, SW46 DOWN, SW47 UP, SW48 RIGHT, SW5 R, SW6 T, SW7 Y, SW8 U, SW9 I, U6 PRTR5V0U2X, Y1 8MHz

Commit message: v2.2
Parts:
- SW25: footprint Laptreus v2 Footprints:Hybrid_Kailh_MX_Choc_Socket_Through_Hole_With_Diode -> Laptreus v2 Footprints:Hybrid_Kailh_MX_Choc_Socket_Through_Hole_With_Diode_No_Diode_Trace
Connections:
- net LED_STRIP_IN is gone; now on net B7-LED-STRIP: JP1.1
Changed lines of the file:
@@
 F 0 "SW25" H 11450 1860 50  0000 C CNN
 F 1 "SHIFT" H 11300 1670 50  0000 C CNN
-F 2 "Laptreus v2 Footprints:Hybrid_Kailh_MX_Choc_Socket_Through_Hole_With_Diode" H 11300 1750 60  0001 C CNN
+F 2 "Laptreus v2 Footprints:Hybrid_Kailh_MX_Choc_Socket_Through_Hole_With_Diode_No_Diode_Trace" H 11300 1750 60  0001 C CNN
 F 3 "" H 11300 1750 60  0001 C CNN
 F 4 "CPG151101S11" H 1000 -1250 50  0001 C CNN "Manufacturer Part Number"
@@
 	4900 6600 4300 6600
 Text Label 3900 3950 2    49   ~ 0
-LED_STRIP_IN
+B7-LED-STRIP
 Wire Wire Line
 	3900 3950 4100 3950
