File: pcb/Laptreus-v2/Laptreus-v2.kicad_pcb (KiCad board)
At the start: 2 copper layers, 286 x 102 mm, 105 parts, among them J1 Conn_01x16, J2 Conn_01x12, SW1 TAB, SW10 O, SW11 P, SW12 BKSP, SW13 ESC, SW14 A, SW15 S, SW16 D, SW17 F/LOWER, SW18 G, SW19 H, SW2 Q, SW20 J/RAISE, SW21 K, SW22 L, SW23 ;, SW24 ", SW25 SHIFT, SW26 Z, SW27 X, SW28 C, SW29 V, SW3 W, SW30 B, SW31 N, SW32 M, SW33 ,, SW34 ., SW35 /, SW36 ENTER, SW37 HYPER, SW38 CTRL/GRV, SW39 ALT/TAB, SW4 E, SW40 CMD, SW41 BKSP/LIFT, SW42 SHIFT, SW43 SPACE, SW44 ENTER/LIFT, SW45 LEFT, SW46 DOWN, SW47 UP, SW48 RIGHT, SW49 SPECIAL, SW5 R, SW50 SPECIAL, SW6 T, SW7 Y, SW8 U, SW9 I, U1 AdafruitFeather32u4BLE

Commit message: Adding first attempts at laptreus v2
Parts:
- removed D24, D25, D36: DIODE, Laptreus v2 Footprints:Diode-dual
- removed J2: Conn_01x12, Connector_PinHeader_2.54mm:PinHeader_1x12_P2.54mm_Vertical
- removed SW12: BKSP, Laptreus v2 Footprints:Hybrid_Kailh_MX_Socket_Through_Hole
- removed SW13: ESC, Laptreus v2 Footprints:Hybrid_Kailh_MX_Socket_Through_Hole
- removed SW24: ", Laptreus v2 Footprints:Hybrid_Kailh_MX_Socket_Through_Hole
- removed SW25: SHIFT, Laptreus v2 Footprints:Hybrid_Kailh_MX_Socket_Through_Hole
- removed SW36: ENTER, Laptreus v2 Footprints:Hybrid_Kailh_MX_Socket_Through_Hole
- added C1: 10µF, Adafruit Feather 32u4 Bluefruit LE:0805-NO, F.Cu at (250.3, 107.6)
- added C2: 1uF, Adafruit Feather 32u4 Bluefruit LE:0805-NO, F.Cu at (270.2, 83.7)
- added C3: 10µF, Adafruit Feather 32u4 Bluefruit LE:0805-NO, F.Cu at (250.4, 103.0)
- added C4: 1uF, Adafruit Feather 32u4 Bluefruit LE:0805-NO, F.Cu at (250.3, 105.3)
- added C5: 10µF, Adafruit Feather 32u4 Bluefruit LE:0805-NO, F.Cu at (217.0, 102.1)
- added C6: 1uF, Adafruit Feather 32u4 Bluefruit LE:0805-NO, F.Cu at (231.9, 100.9)
- added C7: 10uF, Adafruit Feather 32u4 Bluefruit LE:_0805MP, F.Cu at (238.2, 103.6)
- added CHG1: ORANGE, Adafruit Feather 32u4 Bluefruit LE:CHIPLED_0805_NOOUTLINE, F.Cu at (219.3, 90.9)
- added F1: Polyfuse, Keeb_components:R_0805, B.Cu at (105.6, 89.0)
- added FID: FIDUCIAL, hole:FIDUCIAL, B.Cu at (93.8, 162.5)
- added FID: FIDUCIAL, hole:FIDUCIAL, B.Cu at (372.2, 75.1)
- added IC1: ATMEGA32U4-MU, Adafruit Feather 32u4 Bluefruit LE:TQFN44_7MM, F.Cu at (238.2, 98.2)
- added L1: RED, Adafruit Feather 32u4 Bluefruit LE:CHIPLED_0805_NOOUTLINE, F.Cu at (233.1, 87.5)
- added R1: 22, Keeb_components:R_0805, B.Cu at (108.0, 87.8)
- added R1: 1K, Adafruit Feather 32u4 Bluefruit LE:0805-NO, F.Cu at (219.3, 95.0)
- added R10: 2.2K, Adafruit Feather 32u4 Bluefruit LE:0805-NO, F.Cu at (233.1, 91.3)
- added R2: 22, Keeb_components:R_0805, B.Cu at (110.3, 87.8)
- added R2: 100K, Adafruit Feather 32u4 Bluefruit LE:0805-NO, F.Cu at (251.0, 94.0)
- added R3: 5.1k, Keeb_components:R_0805, B.Cu at (105.6, 84.2)
- added R3: 10K\, Adafruit Feather 32u4 Bluefruit LE:0805-NO, F.Cu at (227.5, 96.6)
- added R4: 5.1k, Keeb_components:R_0805, B.Cu at (112.7, 84.2)
- added R4: 100K, Adafruit Feather 32u4 Bluefruit LE:0805-NO, F.Cu at (237.2, 89.7)
- added R5: 100K, Adafruit Feather 32u4 Bluefruit LE:0805-NO, F.Cu at (239.0, 91.7)
- added R6: 2.2K, Adafruit Feather 32u4 Bluefruit LE:0805-NO, F.Cu at (270.7, 81.0)
- added R7: 2.2K, Adafruit Feather 32u4 Bluefruit LE:0805-NO, F.Cu at (270.5, 78.0)
- added S0: DTSM-6, dtsm:KSEM31GLFS, B.Cu at (119.7, 119.7)
- added S1: Screw, footprints:5.5_5x2.5mm, F.Cu at (115.1, 100.0)
- added S2: Screw, footprints:5.5_5x2.5mm, F.Cu at (350.5, 99.4)
- added S3: Screw, footprints:5.5_5x2.5mm, F.Cu at (218.7, 118.6)
- added S4: Screw, footprints:10x5_7x2.5mm, F.Cu at (92.5, 128.3)
- added S5: Screw, footprints:10x5_7x2.5mm, F.Cu at (373.5, 128.3)
- added S6: Screw, footprints:5.5_5x2.5mm, F.Cu at (280.6, 156.7)
- added S7: Tofu screw, footprints:5.5_5x2.5mm, F.Cu at (233.0, 108.9)
- added S8: Tofu screw, footprints:5.5_5x2.5mm, F.Cu at (116.7, 156.9)
- added S9: Tofu screw, footprints:5.5_5x2.5mm, F.Cu at (350.5, 156.9)
- added SW_RESET2: SWITCH_PUSH, Laptreus v2 Footprints:Hybrid_Kailh_MX_Socket_Through_Hole, F.Cu at (252.1, 188.0)
- added TP1: SWCLK, Adafruit Feather 32u4 Bluefruit LE:PAD-1.5X2.0, F.Cu at (250.6, 78.0)
- added TP2: SWDIO, Adafruit Feather 32u4 Bluefruit LE:PAD-1.5X2.0, F.Cu at (250.7, 75.3)
- added TP3: SWDIO, Adafruit Feather 32u4 Bluefruit LE:PAD-1.5X2.0, F.Cu at (250.7, 80.7)
- added U2: USBLC6-2SC6, Keeb_components:USBLC6-2SC6, B.Cu at (109.1, 83.6)
- added U2: SPX3819-3.3, Adafruit Feather 32u4 Bluefruit LE:SOT23-5, F.Cu at (250.7, 98.4)
- added U3: MBT40, Adafruit Feather 32u4 Bluefruit LE:BLE_MODULE_RAYTAC_MDBT40, F.Cu at (260.5, 80.6)
- added X1: JSTPH, Adafruit Feather 32u4 Bluefruit LE:JSTPH2, F.Cu at (222.5, 107.1)
- added Y1: 8MHz, Adafruit Feather 32u4 Bluefruit LE:RESONATOR-SMD, F.Cu at (244.9, 98.7)
- D1: value DIODE -> MBR120; footprint Laptreus v2 Footprints:Diode-dual -> Adafruit Feather 32u4 Bluefruit LE:SOD-123
- D12: value DIODE -> RED; footprint Laptreus v2 Footprints:Diode-dual -> Adafruit Feather 32u4 Bluefruit LE:CHIPLED_0805_NOOUTLINE
- D13: value DIODE -> BLUE; footprint Laptreus v2 Footprints:Diode-dual -> Adafruit Feather 32u4 Bluefruit LE:CHIPLED_0805_NOOUTLINE
- J1: value Conn_01x16 -> HRO-TYPE-C-31-M-12; footprint Connector_PinHeader_2.54mm:PinHeader_1x16_P2.54mm_Vertical -> Keeb_components:HRO-TYPE-C-31-M-12; moved to B.Cu
- SW1: value TAB -> SW_PUSH; footprint Laptreus v2 Footprints:Hybrid_Kailh_MX_Socket_Through_Hole -> Button_Switch_SMD:SW_SPST_TL3342; moved to B.Cu
- SW41: value BKSP/LIFT -> SHIFT
- SW42: value SHIFT -> BKSP/LIFT
- SW43: value SPACE -> ENTER/LIFT
- SW44: value ENTER/LIFT -> SPACE
- U1: value AdafruitFeather32u4BLE -> MCP73831T-2ACI/OT; footprint Laptreus v2 Footprints:Adafruit Feather 32u4 BLE -> Adafruit Feather 32u4 Bluefruit LE:SOT23-5
- moved SW1 242.2 mm to (121.1, 118.8), turned to 180 degrees
- moved D12 165.6 mm to (274.6, 81.1), turned to 270 degrees
- moved D1 144.0 mm to (217.3, 99.9), turned to 0 degrees
- moved J1 116.3 mm to (108.7, 70.5)
- moved D4 109.4 mm to (327.0, 176.5), turned to 180 degrees
- moved D9 107.4 mm to (144.6, 175.4), turned to 180 degrees
- moved D3 104.8 mm to (339.0, 176.5), turned to 180 degrees
- moved D10 103.2 mm to (132.6, 175.5), turned to 180 degrees
- moved D5 101.8 mm to (315.0, 176.5), turned to 180 degrees
- moved D6 101.1 mm to (303.0, 176.5), turned to 180 degrees
- moved D2 100.8 mm to (351.0, 176.5), turned to 180 degrees
- moved D8 99.6 mm to (156.6, 175.4), turned to 180 degrees
- moved D11 99.4 mm to (120.6, 175.5), turned to 180 degrees
- moved D7 98.7 mm to (168.6, 175.4), turned to 180 degrees
- moved D16 95.3 mm to (327.0, 181.5), turned to 180 degrees
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Connections:
- J1 pad 1: /RESET -> (no net)
- J1 pad 10: /COL1 -> (no net)
- J1 pad 11: Net-(J1-Pad11) -> (no net)
- J1 pad 12: Net-(J1-Pad12) -> (no net)
- J1 pad 13: Net-(J1-Pad13) -> (no net)
- J1 pad 2: +5V -> (no net)
- J1 pad 3: Net-(J1-Pad3) -> (no net)
- J1 pad 4: GND -> (no net)
- J1 pad 5: /ROW0 -> (no net)
- J1 pad 6: /ROW1 -> (no net)
- J1 pad 7: /ROW2 -> (no net)
- J1 pad 8: /ROW4 -> (no net)
- J1 pad 9: /ROW3 -> (no net)
- SW1 pad 1: /ROW4 -> (no net)
- SW1 pad 2: Net-(D1-Pad1) -> (no net)
- SW_POW_EN1 pad 2: /Enable -> /EN
- SW_POW_EN1 pad 3: (no net) -> Net-(SW_POW_EN1-Pad3)
- U1 pad 1: (no net) -> Net-(R1-Pad2)
- U1 pad 2: (no net) -> GND
- U1 pad 3: (no net) -> VBAT
- U1 pad 4: (no net) -> VBUS
- U1 pad 5: (no net) -> Net-(R3-Pad1)
Routing:
- net (no net): track 0.00 -> 80.3 mm, vias 0 -> 4
Other:
- board size 286 x 102 mm -> 285 x 94.6 mm

Commit message: switches aligned, leds circled
Parts:
- removed D50: DIODE, Laptreus v2 Footprints:Diode-dual
- removed the R1 at (108.0, 87.8)
- removed the R1 at (219.3, 95.0)
- removed the R2 at (110.3, 87.8)
- removed the R2 at (251.0, 94.0)
- removed the R3 at (105.6, 84.2)
- removed the R3 at (227.5, 96.6)
- removed the R4 at (112.7, 84.2)
- removed the R4 at (237.2, 89.7)
- removed S0: DTSM-6, dtsm:KSEM31GLFS
- removed the U2 at (109.1, 83.6)
- removed the U2 at (250.7, 98.4)
- added C10: 1uF, Adafruit Feather 32u4 Bluefruit LE:_0805MP, F.Cu at (107.8, 275.5)
- added C11: 1uF, Adafruit Feather 32u4 Bluefruit LE:_0805MP, F.Cu at (80.0, 275.4)
- added C12: 1uF, Adafruit Feather 32u4 Bluefruit LE:_0805MP, B.Cu at (80.2, 259.4)
- added C13: 1uF, Adafruit Feather 32u4 Bluefruit LE:_0805MP, B.Cu at (107.8, 259.4)
- added C14: 1uF, Adafruit Feather 32u4 Bluefruit LE:_0805MP, B.Cu at (107.8, 275.5)
- added C15: 1uF, Adafruit Feather 32u4 Bluefruit LE:_0805MP, B.Cu at (80.0, 275.4)
- added C8: 1uF, Adafruit Feather 32u4 Bluefruit LE:_0805MP, F.Cu at (80.2, 259.4)
- added C9: 1uF, Adafruit Feather 32u4 Bluefruit LE:_0805MP, F.Cu at (107.8, 259.4)
- added D24: DIODE, Laptreus v2 Footprints:Diode-dual, F.Cu at (138.1, 181.9)
- added D25: DIODE, Laptreus v2 Footprints:Diode-dual, F.Cu at (330.0, 179.3)
- added D36: DIODE, Laptreus v2 Footprints:Diode-dual, F.Cu at (138.1, 184.4)
- added D55: DIODE, Laptreus v2 Footprints:Diode-dual, F.Cu at (233.0, 196.6)
- added D56: DIODE, Laptreus v2 Footprints:Diode-dual, F.Cu at (214.0, 196.6)
- added D60: RED, Adafruit Feather 32u4 Bluefruit LE:CHIPLED_0805_NOOUTLINE, F.Cu at (332.2, 216.1)
- added D61: BLUE, Adafruit Feather 32u4 Bluefruit LE:CHIPLED_0805_NOOUTLINE, F.Cu at (332.1, 213.0)
- added G***: LOGO, Laptreus v2 Footprints:PlateLayout, F.Cu at (232.8, 162.2)
- added H1: B7, Adafruit NeoPixel Ring 12:1X01-CLEANBIG, F.Cu at (213.0, 226.0)
- added H2: GND, Adafruit NeoPixel Ring 12:1X01-CLEANBIG, F.Cu at (216.0, 226.0)
- added H3: +5v, Adafruit NeoPixel Ring 12:1X01-CLEANBIG, F.Cu at (219.0, 226.0)
- added H4: B0, Adafruit NeoPixel Ring 12:1X01-CLEANBIG, F.Cu at (222.0, 226.0)
- added J2: ISP, Laptreus v2 Footprints:isp_standard, F.Cu at (231.0, 212.0)
- added JP1: PINHD-1X1CB, Adafruit NeoPixel Ring 12:1X01-CLEANBIG, F.Cu at (93.9, 266.2)
- added JP2: PINHD-1X1CB, Adafruit NeoPixel Ring 12:1X01-CLEANBIG, F.Cu at (93.9, 271.9)
- added JP3: PINHD-1X1CB, Adafruit NeoPixel Ring 12:1X01-CLEANBIG, F.Cu at (93.9, 269.1)
- added JP4: PINHD-1X1CB, Adafruit NeoPixel Ring 12:1X01-CLEANBIG, F.Cu at (93.9, 263.3)
- added LED1: WS28115050, Adafruit NeoPixel Ring 12:WS28115050, B.Cu at (85.9, 281.3)
- added LED10: WS28115050, Adafruit NeoPixel Ring 12:WS28115050, F.Cu at (109.9, 267.4)
- added LED11: WS28115050, Adafruit NeoPixel Ring 12:WS28115050, B.Cu at (101.9, 281.3)
- added LED12: WS28115050, Adafruit NeoPixel Ring 12:WS28115050, F.Cu at (101.9, 253.6)
- added LED2: WS28115050, Adafruit NeoPixel Ring 12:WS28115050, F.Cu at (85.9, 253.6)
- added LED3: WS28115050, Adafruit NeoPixel Ring 12:WS28115050, B.Cu at (77.9, 267.4)
- added LED4: WS28115050, Adafruit NeoPixel Ring 12:WS28115050, F.Cu at (77.9, 267.4)
- added LED5: WS28115050, Adafruit NeoPixel Ring 12:WS28115050, B.Cu at (85.9, 253.6)
- added LED6: WS28115050, Adafruit NeoPixel Ring 12:WS28115050, F.Cu at (85.9, 281.3)
- added LED7: WS28115050, Adafruit NeoPixel Ring 12:WS28115050, B.Cu at (101.9, 253.6)
- added LED8: WS28115050, Adafruit NeoPixel Ring 12:WS28115050, F.Cu at (101.9, 281.3)
- added LED9: WS28115050, Adafruit NeoPixel Ring 12:WS28115050, B.Cu at (109.9, 267.4)
- added R1: 1K, Adafruit Feather 32u4 Bluefruit LE:_0805MP, F.Cu at (290.4, 237.6)
- added R11: 5.1k, Adafruit Feather 32u4 Bluefruit LE:0805-NO, B.Cu at (207.1, 57.7)
- added R12: 5.1k, Adafruit Feather 32u4 Bluefruit LE:0805-NO, B.Cu at (200.0, 57.7)
- added R2: 100K, Adafruit Feather 32u4 Bluefruit LE:_0805MP, F.Cu at (323.0, 250.6)
- added R3: 10K\, Adafruit Feather 32u4 Bluefruit LE:_0805MP, F.Cu at (298.8, 236.8)
- added R4: 100K, Adafruit Feather 32u4 Bluefruit LE:_0805MP, F.Cu at (314.3, 246.4)
- added R8: 22, Adafruit Feather 32u4 Bluefruit LE:0805-NO, B.Cu at (202.4, 61.3)
- added R9: 22, Adafruit Feather 32u4 Bluefruit LE:0805-NO, B.Cu at (204.7, 61.3)
- added SW12: BKSP, Laptreus v2 Footprints:Hybrid_Kailh_MX_Socket_Through_Hole, F.Cu at (108.4, 82.0)
- added SW13: ESC, Laptreus v2 Footprints:Hybrid_Kailh_MX_Socket_Through_Hole, F.Cu at (361.1, 100.9)
- added SW24: ", Laptreus v2 Footprints:Hybrid_Kailh_MX_Socket_Through_Hole, F.Cu at (105.1, 100.9)
- added SW25: SHIFT, Laptreus v2 Footprints:Hybrid_Kailh_MX_Socket_Through_Hole, F.Cu at (364.4, 119.7)
- added SW36: ENTER, Laptreus v2 Footprints:Hybrid_Kailh_MX_Socket_Through_Hole, F.Cu at (101.8, 119.6)
- added SW_POW_EN2: SW_SPDT, Laptreus v2 Footprints:EG1218, F.Cu at (157.6, 132.7)
- added U2: SPX3819-3.3, Adafruit Feather 32u4 Bluefruit LE:SOT23-5, F.Cu at (322.7, 255.0)
- added U6: USBLC6-2SC6, Laptreus v2 Footprints:USBLC6-2SC6, B.Cu at (203.5, 57.1)
- C1, C2, C3, C4, C5, C6, R5, R6, R7: footprint Adafruit Feather 32u4 Bluefruit LE:0805-NO -> Adafruit Feather 32u4 Bluefruit LE:_0805MP
- D1: value MBR120 -> DIODE; footprint Adafruit Feather 32u4 Bluefruit LE:SOD-123 -> Laptreus v2 Footprints:Diode-dual
- D12: value RED -> DIODE; footprint Adafruit Feather 32u4 Bluefruit LE:CHIPLED_0805_NOOUTLINE -> Laptreus v2 Footprints:Diode-dual
- D13: value BLUE -> DIODE; footprint Adafruit Feather 32u4 Bluefruit LE:CHIPLED_0805_NOOUTLINE -> Laptreus v2 Footprints:Diode-dual
- D49: value DIODE -> MBR120; footprint Laptreus v2 Footprints:Diode-dual -> Adafruit Feather 32u4 Bluefruit LE:SOD-123
- F1: footprint Keeb_components:R_0805 -> Adafruit Feather 32u4 Bluefruit LE:0805-NO
- J1: footprint Keeb_components:HRO-TYPE-C-31-M-12 -> Laptreus v2 Footprints:HRO-TYPE-C-31-M-12
- R10: value 2.2K -> 10k
- S1, S2, S3, S6, S7, S8, S9: footprint footprints:5.5_5x2.5mm -> Laptreus v2 Footprints:PKRH
- S4, S5: footprint footprints:10x5_7x2.5mm -> Laptreus v2 Footprints:PKRHSL
- SW1: value SW_PUSH -> TAB; footprint Button_Switch_SMD:SW_SPST_TL3342 -> Laptreus v2 Footprints:Hybrid_Kailh_MX_Socket_Through_Hole; moved to F.Cu
- moved SW1 239.6 mm to (357.8, 82.2), turned to 10 degrees
- moved C7 175.3 mm to (305.1, 265.6)
- moved IC1 174.9 mm to (308.1, 258.5)
- moved R5 174.6 mm to (316.1, 248.4)
- moved Y1 174.5 mm to (315.0, 258.5)
- moved C6 173.4 mm to (300.5, 260.1)
- moved C3 172.4 mm to (322.4, 259.6)
- moved C4 172.4 mm to (322.3, 261.9)
- moved C1 172.4 mm to (322.3, 264.2)
- moved D12 168.2 mm to (138.1, 179.4), turned to 180 degrees
- moved TP1 167.1 mm to (325.4, 227.4)
- moved TP2 167.1 mm to (325.5, 224.7)
- moved TP3 167.1 mm to (325.5, 230.1)
- moved L1 161.9 mm to (306.7, 231.7)
- moved R10 161.9 mm to (306.7, 235.5)
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Connections:
- net /MISO renamed MISO
- net /MOSI renamed MOSI
- net /SCK renamed SCK
- D37 pad 2: /COL7 -> /COL11
- D48 pad 2: /COL1 -> /COL0
- F1 pad 1: (no net) -> VCC
- F1 pad 2: (no net) -> VBUS
- IC1 pad 22: Net-(IC1-Pad22) -> /COL11
- IC1 pad 8: Net-(IC1-Pad8) -> /COL0
- J1 pad 1: (no net) -> GND
- J1 pad 10: (no net) -> Net-(J1-Pad10)
- J1 pad 11: (no net) -> VBUS
- J1 pad 12: (no net) -> GND
- J1 pad 13: (no net) -> GND
- J1 pad 2: (no net) -> VBUS
- J1 pad 3: (no net) -> Net-(J1-Pad3)
- J1 pad 4: (no net) -> Net-(J1-Pad4)
- J1 pad 5: (no net) -> D-
- J1 pad 6: (no net) -> D+
- J1 pad 7: (no net) -> D-
- J1 pad 8: (no net) -> D+
- J1 pad 9: (no net) -> Net-(J1-Pad9)
- R10 pad 1: /13 -> GND
- R10 pad 2: Net-(L1-PadA) -> Net-(R10-Pad2)
- R6 pad 2: Net-(D12-PadA) -> Net-(D60-PadA)
- R7 pad 2: Net-(D13-PadA) -> Net-(D61-PadA)
- S1 pad 1: (no net) -> GND
- S2 pad 1: (no net) -> GND
- S3 pad 1: (no net) -> GND
- S4 pad 1: (no net) -> GND
- S5 pad 1: (no net) -> GND
- S6 pad 1: (no net) -> GND
- S7 pad 1: (no net) -> GND
- S8 pad 1: (no net) -> GND
- S9 pad 1: (no net) -> GND
- SW1 pad 1: (no net) -> /ROW0
- SW1 pad 2: (no net) -> Net-(D1-Pad1)
- SW37 pad 1: /ROW4 -> /ROW3
- SW48 pad 1: /ROW4 -> /ROW3
- SW49 pad 2: Net-(D49-Pad1) -> Net-(D55-Pad1)
Routing:
- net (no net): track 80.3 -> 0.00 mm, vias 4 -> 0
- net GND: track 0.00 -> 24.0 mm
- net VBUS: track 0.00 -> 22.6 mm, vias 0 -> 2
- net D+: track 0.00 -> 11.1 mm, vias 0 -> 2
- net D-: track 0.00 -> 7.83 mm
- net Net-(J1-Pad10): track 0.00 -> 5.81 mm
- net Net-(J1-Pad4): track 0.00 -> 5.68 mm
- net /AREF: track 0.00 -> 3.15 mm
- net Net-(R9-Pad1): track 0.00 -> 1.68 mm
- net Net-(R8-Pad2): track 0.00 -> 1.68 mm

Commit message: Starting work on the atmega layout
Parts:
- removed S3: Screw, Laptreus v2 Footprints:PKRH
- added C16: 100nF, Laptreus v2 Footprints:Capacitor-0805MP, F.Cu at (208.4, 80.7)
- C1, C10, C11, C12, C13, C14, C15, C2, C3, C4, C5, C6, C7, C8, C9: footprint Adafruit Feather 32u4 Bluefruit LE:_0805MP -> Laptreus v2 Footprints:Capacitor-0805MP
- F1, R11, R12, R8, R9: footprint Adafruit Feather 32u4 Bluefruit LE:0805-NO -> Laptreus v2 Footprints:0805-NO; moved to F.Cu
- J1, U6: moved to F.Cu
- R1, R2, R3, R4, R5, R6, R7: footprint Adafruit Feather 32u4 Bluefruit LE:_0805MP -> Laptreus v2 Footprints:0805-NO
- R10: footprint Adafruit Feather 32u4 Bluefruit LE:0805-NO -> Laptreus v2 Footprints:0805-NO
- S1: footprint Laptreus v2 Footprints:PKRH -> Laptreus v2 Footprints:PKRH-Round
- SW12: footprint Laptreus v2 Footprints:Hybrid_Kailh_MX_Socket_Through_Hole -> Laptreus v2 Footprints:Hybrid_Kailh_MX_Socket
- TP1, TP2, TP3: moved to B.Cu
- moved TP3 167.8 mm to (248.9, 80.8)
- moved C2 165.9 mm to (238.6, 78.8)
- moved C7 165.8 mm to (232.9, 116.4), turned to 90 degrees
- moved TP1 163.0 mm to (248.8, 83.5)
- moved D60 160.9 mm to (259.7, 72.5)
- moved D61 160.4 mm to (254.7, 72.5)
- moved TP2 158.2 mm to (248.9, 86.2)
- moved Y1 157.8 mm to (226.4, 128.0), turned to 90 degrees
- moved R6 156.4 mm to (257.6, 76.5), turned to 90 degrees
- moved R7 155.3 mm to (254.2, 76.5), turned to 90 degrees
- moved U3 152.6 mm to (247.0, 80.6)
- moved IC1 150.3 mm to (233.0, 128.3), turned to 180 degrees
- moved C6 143.9 mm to (246.5, 126.8), turned to 0 degrees
- moved R11 111.5 mm to (97.4, 77.5), turned to 180 degrees
- moved R12 104.1 mm to (97.4, 75.5), turned to 0 degrees
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Connections:
- F1 pad 1: VCC -> +3V3
- IC1 pad 7: VBUS -> +3V3
- J2 pad 2: VCC -> +3V3
Routing:
- net VBUS: track 22.6 -> 120.4 mm
- net Net-(R8-Pad2): track 1.68 -> 94.9 mm
- net Net-(R9-Pad1): track 1.68 -> 94.9 mm
- net +3V3: track 0.00 -> 66.2 mm
- net Net-(IC1-Pad3): track 0.00 -> 66.1 mm, vias 0 -> 2
- net Net-(IC1-Pad4): track 0.00 -> 65.3 mm
- net GND: track 24.0 -> 75.6 mm, vias 0 -> 5
- net Net-(J1-Pad4): track 5.68 -> 14.2 mm
- net D-: track 7.83 -> 16.2 mm, vias 0 -> 2
- net /MODE: track 0.00 -> 7.49 mm
- net /AREF: track 3.15 -> 9.26 mm
- net Net-(J1-Pad10): track 5.81 -> 10.9 mm
- net D+: track 11.1 -> 16.1 mm
- net Net-(IC1-Pad16): track 0.00 -> 3.54 mm
- net Net-(IC1-Pad17): track 0.00 -> 3.50 mm
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Other:
- net class Default: trace_width 0.25 -> 0.2; via_dia 0.9 -> 0.6; via_drill 0.6 -> 0.4
- net class Ground: trace_width 0.4 -> 0.25
- net class Power: trace_width 0.4 -> 0.25
- net class USB added: clearance 0.2, trace_width 0.2, via_dia 0.6, via_drill 0.4
- rule trace_min: 0.25 -> 0.2
- rule via_min_drill: 0.6 -> 0.4
- rule via_min_size: 0.9 -> 0.6
- board text added: "Red - Mode Blue - Connected"

Commit message: prep for printing v2.1 of the laptre
Parts:
- removed C1: 10µF, Laptreus v2 Footprints:Capacitor-0805MP
- removed C10, C11, C12, C13, C14, C15, C6, C8, C9: 1uF, Laptreus v2 Footprints:Capacitor-0805MP
- removed C16: 100nF, Laptreus v2 Footprints:Capacitor-0805MP
- removed CHG1: ORANGE, Adafruit Feather 32u4 Bluefruit LE:CHIPLED_0805_NOOUTLINE
- removed D49: MBR120, Adafruit Feather 32u4 Bluefruit LE:SOD-123
- removed D55, D56: DIODE, Laptreus v2 Footprints:Diode-dual
- removed D60: RED, Adafruit Feather 32u4 Bluefruit LE:CHIPLED_0805_NOOUTLINE
- removed D61: BLUE, Adafruit Feather 32u4 Bluefruit LE:CHIPLED_0805_NOOUTLINE
- removed FID (x2): FIDUCIAL, hole:FIDUCIAL
- removed G***: LOGO, Laptreus v2 Footprints:PlateLayout
- removed H1: B7, Adafruit NeoPixel Ring 12:1X01-CLEANBIG
- removed H2: GND, Adafruit NeoPixel Ring 12:1X01-CLEANBIG
- removed H3: +5v, Adafruit NeoPixel Ring 12:1X01-CLEANBIG
- removed H4: B0, Adafruit NeoPixel Ring 12:1X01-CLEANBIG
- removed J2: ISP, Laptreus v2 Footprints:isp_standard
- removed JP4: PINHD-1X1CB, Adafruit NeoPixel Ring 12:1X01-CLEANBIG
- removed LED1, LED10, LED11, LED12, LED2, LED3, LED4, LED5, LED6, LED7, LED8, LED9: WS28115050, Adafruit NeoPixel Ring 12:WS28115050
- removed R2, R4, R5: 100K, Laptreus v2 Footprints:0805-NO
- removed R3: 10K\, Laptreus v2 Footprints:0805-NO
- removed R6, R7: 2.2K, Laptreus v2 Footprints:0805-NO
- removed S1: Screw, Laptreus v2 Footprints:PKRH-Round
- removed S2, S6: Screw, Laptreus v2 Footprints:PKRH
- removed S4, S5: Screw, Laptreus v2 Footprints:PKRHSL
- removed S7, S8, S9: Tofu screw, Laptreus v2 Footprints:PKRH
- removed SW49, SW50: SPECIAL, Laptreus v2 Footprints:Hybrid_Kailh_MX_Socket_Through_Hole
- removed SW_POW_EN1, SW_POW_EN2: SW_SPDT, Laptreus v2 Footprints:EG1218
- removed TP1: SWCLK, Adafruit Feather 32u4 Bluefruit LE:PAD-1.5X2.0
- removed TP2, TP3: SWDIO, Adafruit Feather 32u4 Bluefruit LE:PAD-1.5X2.0
- removed U1: MCP73831T-2ACI/OT, Adafruit Feather 32u4 Bluefruit LE:SOT23-5
- removed U2: SPX3819-3.3, Adafruit Feather 32u4 Bluefruit LE:SOT23-5
- removed U3: MBT40, Adafruit Feather 32u4 Bluefruit LE:BLE_MODULE_RAYTAC_MDBT40
- removed X1: JSTPH, Adafruit Feather 32u4 Bluefruit LE:JSTPH2
- added BOARD1: BoardOutline, Laptreus v2 Footprints:60-percent-plus-tofu, F.Cu at (233.0, 118.9)
- added FID1: Fiducial, Laptreus v2 Footprints:FIDUCIAL, F.Cu at (92.8, 74.0)
- added FID2: Fiducial, Laptreus v2 Footprints:FIDUCIAL, F.Cu at (372.7, 163.3)
- added FID3: Fiducial, Laptreus v2 Footprints:FIDUCIAL, B.Cu at (92.8, 74.0)
- added FID4: Fiducial, Laptreus v2 Footprints:FIDUCIAL, B.Cu at (372.7, 163.3)
- added R13: 1K, Laptreus v2 Footprints:0805-NO, F.Cu at (235.4, 139.7)
- C2, C4: value 1uF -> 1µF
- C5: value 10µF -> 1µF
- C7: value 10uF -> 1µF
- F1: footprint Laptreus v2 Footprints:0805-NO -> Fuse:Fuse_1206_3216Metric_Pad1.42x1.75mm_HandSolder
- IC1: value ATMEGA32U4-MU -> ATMEGA32U4; footprint Adafruit Feather 32u4 Bluefruit LE:TQFN44_7MM -> Package_QFP:TQFP-44_10x10mm_P0.8mm
- L1: value RED -> YELLOW; moved to B.Cu
- R10: value 10k -> 1K
- R11, R12: value 5.1k -> 5.1K
- SW1, SW2: footprint Laptreus v2 Footprints:Hybrid_Kailh_MX_Socket_Through_Hole -> Laptreus v2 Footprints:Hybrid_Kailh_MX_Socket_No_Alignment_Pad
- SW10, SW11, SW13, SW14, SW15, SW16, SW17, SW18, SW19, SW20, SW21, SW22, SW23, SW24, SW25, SW26, SW27, SW28, SW29, SW3, SW30, SW31, SW32, SW33, SW34, SW35, SW36, SW37, SW38, SW39, SW4, SW40, SW41, SW42, SW43, SW44, SW45, SW46, SW47, SW48, SW5, SW6, SW7, SW8, SW9, SW_RESET2: footprint Laptreus v2 Footprints:Hybrid_Kailh_MX_Socket_Through_Hole -> Laptreus v2 Footprints:Hybrid_Kailh_MX_Socket_Through_Hole_No_Alignment_Pad
- SW12: footprint Laptreus v2 Footprints:Hybrid_Kailh_MX_Socket -> Laptreus v2 Footprints:Hybrid_Kailh_MX_Socket_Through_Hole_No_Alignment_Pad
- SW_RESET1: moved to B.Cu
- U6: value USBLC6-2SC6 -> PRTR5V0U2X; footprint Laptreus v2 Footprints:USBLC6-2SC6 -> Laptreus v2 Footprints:SOT143B
- moved R11 270.8 mm to (368.2, 73.6), turned to 0 degrees
- moved R12 270.8 mm to (368.2, 76.7), turned to 180 degrees
- moved J1 248.6 mm to (357.3, 69.8)
- moved U6 224.7 mm to (343.2, 75.0), turned to 180 degrees
- moved JP1 185.1 mm to (213.0, 124.5), turned to 90 degrees
- moved JP3 185.0 mm to (213.0, 127.5), turned to 90 degrees
- moved JP2 184.9 mm to (213.0, 130.4), turned to 90 degrees
- moved C3 156.6 mm to (242.8, 124.7), turned to 270 degrees
- moved C4 152.4 mm to (242.8, 131.9), turned to 90 degrees
- moved R1 145.2 mm to (238.4, 102.0), turned to 0 degrees
- moved F1 134.7 mm to (346.9, 75.0), turned to 90 degrees
- moved C5 129.2 mm to (222.6, 122.0), turned to 270 degrees
- moved R8 126.5 mm to (338.7, 73.9), turned to 0 degrees
- moved R9 126.5 mm to (338.7, 76.1), turned to 180 degrees
- moved L1 124.1 mm to (233.0, 131.8), turned to 90 degrees
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Connections:
- net Net-(IC1-Pad16) renamed /XTAL2
- net Net-(IC1-Pad17) renamed /XTAL1
- net Net-(IC1-Pad3) renamed /DR-
- net Net-(IC1-Pad4) renamed /DR+
- C2 pad 1: +3V3 -> +5V
- C3 pad 1: +3V3 -> +5V
- C4 pad 1: +3V3 -> +5V
- C5 pad 1: VBAT -> +5V
- C7 pad 1: +3V3 -> /UCAP
- F1 pad 1: +3V3 -> +5V
- F1 pad 2: VBUS -> +5VRAW
- IC1 pad 1: /7_BLE_IRQ -> (no net)
- IC1 pad 10: MOSI -> (no net)
- IC1 pad 11: MISO -> (no net)
- IC1 pad 12: /COL9 -> B7-LED-STRIP
- IC1 pad 14: +3V3 -> +5V
- IC1 pad 19: /COL5 -> /COL3
- IC1 pad 2: Net-(IC1-Pad2) -> +5V
- IC1 pad 21: /COL3 -> /COL1
- IC1 pad 22: /COL11 -> /COL0
- IC1 pad 24: +3V3 -> +5V
- IC1 pad 25: /4_SWDIO/RST -> /COL5
- IC1 pad 26: /COL10 -> /ROW0
- IC1 pad 27: /COL7 -> /ROW1
- IC1 pad 28: /8_BLE_CS -> (no net)
- IC1 pad 29: /9 -> (no net)
- IC1 pad 30: /COL8 -> /ROW2
- IC1 pad 31: /COL6 -> /ROW3
- IC1 pad 32: /13 -> /C7-13
- IC1 pad 33: +3V3 -> /HWB
- IC1 pad 34: +3V3 -> +5V
- IC1 pad 36: /ROW0 -> /COL11
- IC1 pad 37: /ROW1 -> /COL10
- IC1 pad 38: /ROW2 -> /COL9
- IC1 pad 39: /ROW4 -> /COL8
- IC1 pad 40: /ROW3 -> /COL7
- IC1 pad 41: /COL1 -> /COL6
- IC1 pad 42: /AREF -> (no net)
- IC1 pad 44: +3V3 -> +5V
- IC1 pad 6: +3V3 -> /UCAP
- IC1 pad 7: +3V3 -> +5V
- IC1 pad 8: /COL0 -> (no net)
- IC1 pad 9: SCK -> (no net)
- J1 pad 11: VBUS -> +5VRAW
- J1 pad 2: VBUS -> +5VRAW
- J1 pad 3: Net-(J1-Pad3) -> (no net)
- J1 pad 9: Net-(J1-Pad9) -> (no net)
- JP1 pad 1: +3V3 -> B7-LED-STRIP
- JP2 pad 1: Net-(JP2-Pad1) -> GND
- JP3 pad 1: GND -> +5V
- R1 pad 1: Net-(CHG1-PadC) -> /RESET
- R1 pad 2: Net-(R1-Pad2) -> +5V
- R10 pad 2: Net-(R10-Pad2) -> /HWB
- R8 pad 2: Net-(R8-Pad2) -> D+
- R9 pad 1: Net-(R9-Pad1) -> D-
- U6 pad 1: D+ -> GND
- U6 pad 2: GND -> D+
- U6 pad 4: Net-(R9-Pad1) -> +5V
Routing:
- net GND: track 75.6 -> 738.1 mm, vias 5 -> 9
- net /ROW0: track 0.00 -> 395.2 mm, vias 0 -> 2
- net /ROW1: track 0.00 -> 354.8 mm, vias 0 -> 6
- net /ROW2: track 0.00 -> 309.8 mm, vias 0 -> 6
- net /COL10: track 0.00 -> 298.7 mm, vias 0 -> 1
- net /ROW3: track 0.00 -> 297.2 mm, vias 0 -> 6
- net /COL11: track 0.00 -> 249.1 mm, vias 0 -> 1
- net /COL0: track 0.00 -> 220.3 mm, vias 0 -> 1
- net +5V: track 0.00 -> 204.0 mm, vias 0 -> 7
- net /COL1: track 0.00 -> 203.7 mm, vias 0 -> 1
- net /COL9: track 0.00 -> 201.6 mm, vias 0 -> 1
- net /COL2: track 0.00 -> 187.0 mm, vias 0 -> 1
- net /COL8: track 0.00 -> 185.0 mm, vias 0 -> 1
- net /COL3: track 0.00 -> 170.3 mm, vias 0 -> 1
- net /COL7: track 0.00 -> 157.0 mm, vias 0 -> 1
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- added copper zone on B.Cu, net +5V
- removed copper zone on B.Cu, net GND
Other:
- board size 285 x 94.6 mm -> 285 x 95.1 mm
- net class Default: clearance 0.2 -> 0.16; trace_width 0.2 -> 0.16
- net class Ground: clearance 0.25 -> 0.16; via_dia 0.9 -> 0.6; via_drill 0.6 -> 0.4
- net class Power: clearance 0.25 -> 0.16; via_dia 0.9 -> 0.6; via_drill 0.6 -> 0.4
- net class USB: clearance 0.2 -> 0.1; trace_width 0.2 -> 0.16
- rule pad_to_mask_clearance: 0.2 -> 0.1
- rule solder_mask_min_width: 0.25 -> 0.1
- rule trace_clearance: 0.2 -> 0.16
- rule trace_min: 0.2 -> 0.1
- board text added: "+5V"
- board text added: "1Ah (51x34x5.9)"
- board text added: "400mAh (27x37x5)"
- board text added: "B7"
- board text added: "GND"
- board text added: "JLCJLCJLCJLC"
- board text added: "Laptreus v2.1"
- board text removed: "Laptreus v2.0"
- board text removed: "Red - Mode Blue - Connected"
