File: pcb/Laptreus-v2/Laptreus-v2.kicad_pcb (KiCad board)
At the start: 2 copper layers, 285 x 95.1 mm, 124 parts, among them IC1 ATMEGA32U4, J1 HRO-TYPE-C-31-M-12, SW1 TAB, SW10 O, SW11 P, SW12 BKSP, SW13 ESC, SW14 A, SW15 S, SW16 D, SW17 F/LOWER, SW18 G, SW19 H, SW2 Q, SW20 J/RAISE, SW21 K, SW22 L, SW23 ;, SW24 ", SW25 SHIFT, SW26 Z, SW27 X, SW28 C, SW29 V, SW3 W, SW30 B, SW31 N, SW32 M, SW33 ,, SW34 ., SW35 /, SW36 ENTER, SW37 HYPER, SW38 CTRL/GRV, SW39 ALT/TAB, SW4 E, SW40 CMD, SW41 SHIFT, SW42 BKSP/LIFT, SW43 ENTER/LIFT, SW44 SPACE, SW45 LEFT, SW46 DOWN, SW47 UP, SW48 RIGHT, SW5 R, SW6 T, SW7 Y, SW8 U, SW9 I, U6 PRTR5V0U2X, Y1 8MHz

Commit message: v2.2
Parts:
- D1, D10, D11, D12, D13, D14, D15, D16, D17, D18, D19, D2, D20, D21, D22, D23, D24, D25, D26, D27, D28, D29, D3, D30, D31, D32, D33, D34, D35, D36, D37, D38, D39, D4, D40, D41, D42, D43, D44, D45, D46, D47, D48, D5, D6, D7, D8, D9: footprint Laptreus v2 Footprints:Diode-dual -> Laptreus v2 Footprints:Diode-0805
- SW1, SW2: footprint Laptreus v2 Footprints:Hybrid_Kailh_MX_Socket_No_Alignment_Pad -> Laptreus v2 Footprints:Kailh_Socket_With_Diode_No_Diode_Trace
- SW10, SW11, SW12, SW13, SW15, SW16, SW17, SW18, SW19, SW20, SW21, SW22, SW26, SW27, SW28, SW29, SW3, SW30, SW31, SW32, SW33, SW34, SW35, SW37, SW38, SW39, SW4, SW40, SW41, SW42, SW43, SW44, SW45, SW46, SW47, SW48, SW5, SW6, SW7, SW8, SW9: footprint Laptreus v2 Footprints:Hybrid_Kailh_MX_Socket_Through_Hole_No_Alignment_Pad -> Laptreus v2 Footprints:Hybrid_Kailh_MX_Choc_Socket_Through_Hole_With_Diode
- SW14, SW23, SW24, SW25, SW36: footprint Laptreus v2 Footprints:Hybrid_Kailh_MX_Socket_Through_Hole_No_Alignment_Pad -> Laptreus v2 Footprints:Hybrid_Kailh_MX_Choc_Socket_Through_Hole_With_Diode_No_Diode_Trace
- SW_RESET2: footprint Laptreus v2 Footprints:Hybrid_Kailh_MX_Socket_Through_Hole_No_Alignment_Pad -> Laptreus v2 Footprints:Kailh_Socket_With_Diode_No_Diode_Trace
- U6: footprint Laptreus v2 Footprints:SOT143B -> Package_TO_SOT_SMD:SOT-143_Handsoldering
- moved D41 18.4 mm to (264.6, 159.3)
- moved D14 17.4 mm to (332.8, 95.9), turned to 100 degrees
- moved D24 16.7 mm to (97.9, 93.7), turned to 80 degrees
- moved D2 14.8 mm to (330.0, 80.0), turned to 100 degrees
- moved D36 13.6 mm to (93.4, 119.5), turned to 80 degrees
- moved D13 12.1 mm to (371.4, 101.2), turned to 100 degrees
- moved D43 11.4 mm to (207.9, 139.0), turned to 47.5 degrees
- moved D1 11.2 mm to (368.3, 84.1), turned to 100 degrees
- moved D12 11.0 mm to (100.0, 82.0), turned to 80 degrees
- moved D19 11.0 mm to (191.6, 111.0), turned to 80 degrees
- moved D6 11.0 mm to (255.1, 95.1), turned to 100 degrees
- moved D10 11.0 mm to (138.6, 82.4), turned to 80 degrees
- moved D33 11.0 mm to (151.3, 120.1), turned to 80 degrees
- moved D27 11.0 mm to (318.0, 122.7), turned to 100 degrees
- moved D29 11.0 mm to (280.5, 129.4), turned to 100 degrees
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Connections:
- net B7-LED-STRIP renamed /B7-LED-STRIP
Routing:
- net GND: track 738.1 -> 275.1 mm, vias 9 -> 47
- net /COL10: track 298.7 -> 213.8 mm, vias 1 -> 2
- net /ROW2: track 309.8 -> 369.2 mm, vias 6 -> 8
- net /ROW1: track 354.8 -> 407.3 mm, vias 6 -> 8
- net /ROW0: track 395.2 -> 439.4 mm, vias 2 -> 6
- net /COL5: track 111.2 -> 141.2 mm, vias 1 -> 2
- net /ROW3: track 297.2 -> 320.8 mm, vias 6 -> 8
- net Net-(D24-Pad1): track 9.71 -> 32.6 mm
- net /RESET: track 58.0 -> 78.7 mm, vias 2 -> 1
- net /COL4: track 148.9 -> 169.1 mm, vias 1 -> 2
- net Net-(D23-Pad1): track 9.01 -> 27.0 mm
- net Net-(D36-Pad1): track 5.84 -> 19.8 mm, vias 0 -> 1
- net /COL11: track 249.1 -> 236.3 mm, vias 1 -> 2
- net Net-(D14-Pad1): track 8.40 -> 20.4 mm, vias 0 -> 1
- net /COL1: track 203.7 -> 215.2 mm, vias 1 -> 2
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- added copper zone on B.Cu, net GND
Other:
- board text added: "Laptreus v2.2"
- board text removed: "Laptreus v2.1"

Commit message: v2.3 of shapeshifter 4060, also plate
Parts:
- added J2: Conn_01x04, Connector_JST:JST_SH_SM04B-SRSS-TB_1x04-1MP_P1.00mm_Horizontal, F.Cu at (368.0, 74.8)
- added J3: Conn_01x04_Female, Connector_PinHeader_1.00mm:PinHeader_1x04_P1.00mm_Vertical, F.Cu at (369.5, 80.8)
- added J4: Conn_01x04_Female, Connector_PinHeader_1.00mm:PinHeader_1x04_P1.00mm_Vertical, F.Cu at (369.5, 78.9)
- added KittyB: Val**, Laptreus v2 Footprints:Kitty, B.Cu at (101.5, 156.9)
- added KittyF: Val**, Laptreus v2 Footprints:Kitty, F.Cu at (101.0, 156.9)
- D1, D10, D11, D12, D13, D14, D15, D16, D17, D18, D19, D2, D20, D21, D22, D23, D24, D25, D26, D27, D28, D29, D3, D30, D31, D32, D33, D34, D35, D36, D37, D38, D39, D4, D40, D41, D42, D43, D44, D45, D46, D47, D48, D5, D6, D7, D8, D9: footprint Laptreus v2 Footprints:Diode-0805 -> Laptreus v2 Footprints:D_SOD-323_With_Adhesive
- F1: footprint Fuse:Fuse_1206_3216Metric_Pad1.42x1.75mm_HandSolder -> Laptreus v2 Footprints:Fuse_1812_4532Metric_With_Adhesive
- IC1: footprint Package_QFP:TQFP-44_10x10mm_P0.8mm -> Laptreus v2 Footprints:TQFP-44_10x10mm_P0.8mm
- L1: footprint Adafruit Feather 32u4 Bluefruit LE:CHIPLED_0805_NOOUTLINE -> LED_SMD:LED_0603_1608Metric_Castellated
- R1, R10, R11, R12, R13, R8, R9: footprint Laptreus v2 Footprints:0805-NO -> Laptreus v2 Footprints:R_0603_1608Metric_With_Adhesive
- SW2: footprint Laptreus v2 Footprints:Kailh_Socket_With_Diode_No_Diode_Trace -> Laptreus v2 Footprints:Hybrid_Kailh_MX_Choc_Socket_Through_Hole_With_Diode
- U6: footprint Package_TO_SOT_SMD:SOT-143_Handsoldering -> Laptreus v2 Footprints:SOT-143_With_Adhesive
- moved L1 47.2 mm to (221.2, 93.8), turned to 0 degrees
- moved R13 43.2 mm to (229.4, 96.9), turned to 0 degrees
- moved R11 9.27 mm to (372.2, 82.0)
- moved R12 8.47 mm to (372.2, 84.2)
- moved R9 8.19 mm to (346.3, 75.2)
- moved R8 8.07 mm to (346.3, 73.6)
- moved SW_RESET1 7.50 mm to (233.0, 81.7)
- moved U6 6.78 mm to (349.7, 74.4)
- moved D2 5.04 mm to (330.8, 85.0), turned to 280 degrees
- moved F1 4.79 mm to (349.1, 80.5), turned to 270 degrees
- moved R10 1.53 mm to (236.2, 139.7)
- moved D39 0.25 mm to (303.0, 147.7), turned to 280 degrees
- moved D15 0.25 mm to (314.6, 103.8), turned to 280 degrees
- moved D16 0.25 mm to (295.3, 104.0), turned to 280 degrees
- moved D29 0.25 mm to (280.3, 129.2), turned to 280 degrees
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Connections:
- R13 pad 1: Net-(L1-PadA) -> Net-(L1-Pad2)
Routing:
- net /C7-13: track 5.07 -> 66.9 mm, vias 0 -> 2
- net Net-(D2-Pad1): track 19.6 -> 0.00 mm
- net +5VRAW: track 18.3 -> 34.0 mm, vias 0 -> 5
- net GND: track 275.1 -> 260.9 mm, vias 47 -> 48
- net D+: track 25.8 -> 35.7 mm
- net /DR-: track 144.0 -> 153.2 mm
- net /DR+: track 144.5 -> 153.1 mm
- net Net-(J1-Pad10): track 13.8 -> 22.2 mm
- net Net-(L1-Pad2): track 0.00 -> 7.92 mm, vias 0 -> 1
- net +5V: track 201.6 -> 208.8 mm, vias 7 -> 9
- net D-: track 25.7 -> 32.8 mm
- net Net-(J1-Pad4): track 13.3 -> 19.9 mm
- net /RESET: track 78.7 -> 72.3 mm
- net Net-(L1-PadA): track 4.97 -> 0.00 mm, vias 1 -> 0
- net /COL10: track 213.8 -> 210.4 mm
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- removed copper zone on B.Cu, net +5V
- removed copper zone on B.Cu, net GND
- removed copper zone on F.Cu, net GND
Other:
- board text added: "G+-V"
- board text added: "Laptreus v2.3"
- board text removed: "Laptreus v2.2"
