File: pcb/Laptreus-v2/Laptreus-v2.kicad_pcb (KiCad board)
At the start: 2 copper layers, 285 x 95.1 mm, 129 parts, among them IC1 ATMEGA32U4, J1 HRO-TYPE-C-31-M-12, J2 Conn_01x04, J3 Conn_01x04_Female, J4 Conn_01x04_Female, SW1 TAB, SW10 O, SW11 P, SW12 BKSP, SW13 ESC, SW14 A, SW15 S, SW16 D, SW17 F/LOWER, SW18 G, SW19 H, SW2 Q, SW20 J/RAISE, SW21 K, SW22 L, SW23 ;, SW24 ", SW25 SHIFT, SW26 Z, SW27 X, SW28 C, SW29 V, SW3 W, SW30 B, SW31 N, SW32 M, SW33 ,, SW34 ., SW35 /, SW36 ENTER, SW37 HYPER, SW38 CTRL/GRV, SW39 ALT/TAB, SW4 E, SW40 CMD, SW41 SHIFT, SW42 BKSP/LIFT, SW43 ENTER/LIFT, SW44 SPACE, SW45 LEFT, SW46 DOWN, SW47 UP, SW48 RIGHT, SW5 R, SW6 T, SW7 Y, SW8 U, SW9 I, U6 PRTR5V0U2X, Y1 8MHz

Commit message: Update to remove jst-sh connector
Routing:
- net GND: track 260.9 -> 267.7 mm, vias 48 -> 51
- added copper zone on B.Cu, net +5V
- added copper zone on B.Cu, net GND
- added copper zone on F.Cu, net GND
Changed lines of the file:
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@@
-(kicad_pcb (version 20171130) (host pcbnew "(6.0.0-rc1-dev-1469-g932b9a334)")
+(kicad_pcb (version 20171130) (host pcbnew "(5.1.5-0-10_14)")
   (general
     (thickness 1.6)
     (drawings 42)
-    (tracks 1380)
+    (tracks 1390)
     (zones 0)
     (modules 129)
@@
     (38 B.Mask user)
     (39 F.Mask user)
-    (40 Dwgs.User user)
-    (41 Cmts.User user)
-    (42 Eco1.User user)
-    (43 Eco2.User user)
+    (40 Dwgs.User user hide)
+    (41 Cmts.User user hide)
+    (42 Eco1.User user hide)
+    (43 Eco2.User user hide)
     (44 Edge.Cuts user)
-    (45 Margin user)
-    (46 B.CrtYd user)
-    (47 F.CrtYd user)
-    (48 B.Fab user)
-    (49 F.Fab user)
+    (45 Margin user hide)
+    (46 B.CrtYd user hide)
+    (47 F.CrtYd user hide)
+    (48 B.Fab user hide)
+    (49 F.Fab user hide)
   )
   (setup
@@
     (user_trace_width 0.25)
     (trace_clearance 0.16)
-    (zone_clearance 0.4)
+    (zone_clearance 0.307299)
     (zone_45_only no)
     (trace_min 0.1)
@@
   (segment (start 220.24966 121.769781) (end 215.24966 121.769782) (width 0.25) (layer F.Cu) (net 43))
   (segment (start 213.299645 123.719796) (end 213.299645 124.270054) (width 0.25) (layer F.Cu) (net 43) (status 30))
+  (segment (start 221.399645 127.920052) (end 221.39917 127.919577) (width 0.25) (layer F.Cu) (net 43))
+  (segment (start 222.499645 127.920052) (end 221.399645 127.920052) (width 0.25) (layer F.Cu) (net 43))
+  (segment (start 221.39917 127.919577) (end 221.223644 127.919577) (width 0.25) (layer F.Cu) (net 43))
+  (segment (start 221.223644 127.919577) (end 220.89917 127.595103) (width 0.25) (layer F.Cu) (net 43))
+  (segment (start 220.89917 127.595103) (end 220.89917 125.995103) (width 0.25) (layer F.Cu) (net 43))
+  (segment (start 221.749492 125.144781) (end 224.04966 125.144781) (width 0.25) (layer F.Cu) (net 43))
+  (segment (start 220.89917 125.995103) (end 221.749492 125.144781) (width 0.25) (layer F.Cu) (net 43))
+  (via (at 333.19917 80.995103) (size 0.6) (drill 0.4) (layers F.Cu B.Cu) (net 43))
+  (via (at 234.59917 137.395103) (size 0.6) (drill 0.4) (layers F.Cu B.Cu) (net 43))
+  (via (at 231.39917 137.395103) (size 0.6) (drill 0.4) (layers F.Cu B.Cu) (net 43))
   (segment (start 246.68354 150.844244) (end 246.966583 151.127287) (width 0.16) (layer F.Cu) (net 55) (status 10))
   (segment (start 246.966583 151.127287) (end 246.966583 151.187516) (width 0.16) (layer F.Cu) (net 55))
@@
   (segment (start 368.52417 78.920103) (end 368.52417 76.795103) (width 0.16) (layer F.Cu) (net 84))
   (segment (start 369.52417 78.920103) (end 369.52417 76.795103) (width 0.16) (layer F.Cu) (net 85))
+  (zone (net 0) (net_name "") (layers F&B.Cu) (hatch edge 0.508)
+    (connect_pads (clearance 0.307299))
+    (min_thickness 0.254)
+    (keepout (tracks allowed) (vias allowed) (copperpour not_allowed))
+    (fill (arc_segments 16) (thermal_gap 0.508) (thermal_bridge_width 0.508))
+    (polygon
+      (pts
+        (xy 90.47417 71.495102) (xy 90.49917 76.270103) (xy 245.89917 76.282324) (xy 245.89917 77.395103) (xy 247.87417 77.395103)
+        (xy 247.87417 76.282714) (xy 351.62417 76.295103) (xy 351.62417 71.495102)
+      )
+    )
+  )
+  (zone (net 0) (net_name "") (layers F&B.Cu) (hatch edge 0.508)
+    (connect_pads (clearance 0.4))
+    (min_thickness 0.254)
+    (keepout (tracks not_allowed) (vias not_allowed) (copperpour allowed))
+    (fill (arc_segments 16) (thermal_gap 0.508) (thermal_bridge_width 0.508))
+    (polygon
+      (pts
+        (xy 241.899169 158.995103) (xy 241.899171 158.995104) (xy 241.89917 163.937617) (xy 373.038928 163.937616) (xy 373.038928 147.937616)
+        (xy 376.038928 147.937617) (xy 376.038928 166.937616) (xy 90.038928 166.937616) (xy 90.038928 163.937617) (xy 224.39917 163.937616)
+        (xy 224.39917 158.995102) (xy 236.065839 158.995104) (xy 241.89917 158.995102)
+      )
+    )
+  )
+  (zone (net 43) (net_name GND) (layer F.Cu) (hatch edge 0.508)
+    (connect_pads (clearance 0.307299))
+    (min_thickness 0.254)
+    (fill yes (arc_segments 16) (thermal_gap 0.508) (thermal_bridge_width 0.508))
+    (polygon
+      (pts
+        (xy 376.99917 79.795103) (xy 376.999171 167.495103) (xy 88.999171 167.495102) (xy 88.99917 70.495103) (xy 240.799171 70.495102)
+        (xy 253.099172 70.495103) (xy 351.64917 70.495103) (xy 351.64917 79.795103)
+      )
+    )
+    (polygon
+      (pts
+        (xy 220.545692 120.197748) (xy 220.54569 135.997747) (xy 240.445691 135.997746) (xy 240.445691 120.197746)
+      )
+    )
+  )
+  (zone (net 43) (net_name GND) (layer B.Cu) (hatch edge 0.508)
+    (connect_pads (clearance 0.307299))
+    (min_thickness 0.254)
+    (fill yes (arc_segments 16) (thermal_gap 0.508) (thermal_bridge_width 0.508))
+    (polygon
+      (pts
+        (xy 376.999171 167.495103) (xy 88.999171 167.495102) (xy 88.99917 70.495102) (xy 376.99917 70.495103)
+      )
+    )
+    (polygon
+      (pts
+        (xy 220.545692 120.197748) (xy 220.54569 135.997747) (xy 240.445691 135.997746) (xy 240.445691 120.197746)
+      )
+    )
+  )
+  (zone (net 71) (net_name +5V) (layer B.Cu) (hatch edge 0.508)
+    (connect_pads (clearance 0.307299))
+    (min_thickness 0.254)
+    (fill yes (arc_segments 16) (thermal_gap 0.508) (thermal_bridge_width 0.508) (smoothing chamfer))
+    (polygon
+      (pts
+        (xy 228.445691 121.497746) (xy 237.645692 121.497745) (xy 237.645692 123.697745) (xy 239.845692 123.697745) (xy 239.845692 132.997746)
+        (xy 237.645692 132.997748) (xy 237.645692 135.197748) (xy 228.345691 135.197746) (xy 228.345691 132.997746) (xy 226.145691 132.997746)
+        (xy 226.145691 123.995104) (xy 228.445691 123.995103)
+      )
+    )
+  )
+  (zone (net 43) (net_name GND) (layer F.Cu) (hatch edge 0.508)
+    (connect_pads (clearance 0.307299))
+    (min_thickness 0.254)
+    (fill yes (arc_segments 16) (thermal_gap 0.508) (thermal_bridge_width 0.508) (smoothing chamfer))
+    (polygon
+      (pts
+        (xy 228.445691 121.497746) (xy 237.645692 121.497745) (xy 237.645692 123.697745) (xy 239.845692 123.697745) (xy 239.845692 132.997746)
+        (xy 237.645692 132.997748) (xy 237.645692 135.197748) (xy 228.345691 135.197746) (xy 228.345691 132.997746) (xy 226.145691 132.997746)
+        (xy 226.145691 123.697746) (xy 228.445691 123.697746)
+      )
+    )
+  )
 )
